Commit message: Updating to include real STL meshes

File: src/servo/urdf/servo.urdf (robot description, URDF)
Before this commit: robot servo, 2 links, 1 joints
Links:
- link body: geometry collision box size=.040 .020 .038; visual mesh filename=package://servo/meshes/Servo.stl
- link horn: geometry collision box size=.040 .005 .001; visual mesh filename=package://servo/meshes/ServoHorn.stl
Joints:
- joint swivel: origin xyz=0.15 0 0.4 -> xyz=-0.015 0 0.02

Commit message: Updating to line up STL servo parts correctly

File: src/servo/urdf/servo.urdf (robot description, URDF)
Before this commit: robot servo, 2 links, 1 joints
Links:
- link horn: geometry collision box size=.0413 .0135 .00213; visual mesh filename=package://servo/meshes/ServoHorn.stl
Joints:
- joint swivel: origin xyz=-0.015 0 0.02 -> xyz=-0.01035 0 0.02539

Commit message: Fixing gap between horn and body

File: src/servo/urdf/servo.urdf (robot description, URDF)
Before this commit: robot servo, 2 links, 1 joints
Joints:
- joint swivel: origin xyz=-0.01035 0 0.02539 -> xyz=-0.01035 0 0.0292

Commit message: Adding LeftHip

File: src/servo/urdf/servo.urdf (robot description, URDF)
Before this commit: robot servo, 2 links, 1 joints
Links:
- removed link body
- added link left_hip, mass 1; collision box size=.0625 .0423 .0697; visual mesh filename=package://servo/meshes/LeftHip_V15.stl scale=0.001 0.001 0.001
- added link servo_base, mass 1; collision box size=.040 .020 .038; visual mesh filename=package://servo/meshes/Servo.stl
Joints:
- added joint hip_servo: type fixed, parent left_hip, child servo_base, origin xyz=-0.01035 0 0.0292, axis 0 0 1
- joint swivel: parent body -> servo_base

Commit message: Updating to operate servo in terms of +-90 degree commands

File: src/servo/urdf/servo.urdf (robot description, URDF)
Before this commit: robot servo, 3 links, 2 joints
Joints:
- joint hip_servo: origin xyz=-0.01035 0 0.0292 -> xyz=0 0 0
- joint swivel: origin xyz=-0.01035 0 0.0292 -> xyz=-0.01035 -0.00995 0.0292

Commit message: Updating to get Servo Horn orientation correct

File: src/servo/urdf/servo.urdf (robot description, URDF)
Before this commit: robot servo, 3 links, 2 joints
Joints:
- joint swivel: axis 0 0 1 -> 0 0 -1

Commit message: Initial attempts to get second servo in place (WIP)

File: src/servo/urdf/servo.urdf (robot description, URDF)
Before this commit: robot servo, 3 links, 2 joints
Links:
- removed link horn
- removed link servo_base
- added link left_front_pitch_servo_base, mass 1; collision box size=.040 .020 .038; visual mesh filename=package://servo/meshes/Servo.stl
- added link left_front_pitch_servo_horn, mass 1; collision box size=.0413 .0135 .00213; visual mesh filename=package://servo/meshes/ServoHorn.stl
- added link left_front_yaw_servo_base, mass 1; collision box size=.040 .020 .038; visual mesh filename=package://servo/meshes/Servo.stl
- added link left_front_yaw_servo_horn, mass 1; collision box size=.0413 .0135 .00213; visual mesh filename=package://servo/meshes/ServoHorn.stl
Joints:
- removed joint hip_servo
- added joint hip_pitch_servo: type fixed, parent left_hip, child left_front_pitch_servo_base, origin xyz=0 0 0, axis 0 0 1
- added joint hip_yaw_servo: type fixed, parent left_hip, child left_front_yaw_servo_base, origin xyz=0 0 0, axis 0 0 1
- added joint left_front_pitch_swivel: type continuous, parent left_front_pitch_servo_base, child left_front_pitch_servo_horn, origin xyz=0 0 0, axis 0 0 -1
- joint swivel: child horn -> left_front_yaw_servo_horn; parent servo_base -> left_front_yaw_servo_base

Commit message: Removing Collision and Inertia tgs from URDF until I get it working

File: src/servo/urdf/servo.urdf (robot description, URDF)
Before this commit: robot servo, 5 links, 4 joints
Links:
- link left_front_pitch_servo_base: mass 1 -> None; geometry visual mesh filename=package://servo/meshes/Servo.stl
- link left_front_pitch_servo_horn: mass 1 -> None; geometry visual mesh filename=package://servo/meshes/ServoHorn.stl
- link left_front_yaw_servo_base: mass 1 -> None; geometry visual mesh filename=package://servo/meshes/Servo.stl
- link left_front_yaw_servo_horn: mass 1 -> None; geometry visual mesh filename=package://servo/meshes/ServoHorn.stl
- link left_hip: mass 1 -> None; geometry visual mesh filename=package://servo/meshes/LeftHip_V15.stl scale=0.001 0.001 0.001
Joints:
- joint hip_pitch_servo: axis 0 0 1 -> (none)
- joint hip_yaw_servo: axis 0 0 1 -> (none)
- joint left_front_pitch_swivel: origin xyz=0 0 0 -> xyz=-0.01035 -0.00995 0.0292

Commit message: Sorted out hip pitch and yaw servos and horns... Whew...

File: src/servo/urdf/servo.urdf (robot description, URDF)
Before this commit: robot servo, 5 links, 4 joints
Joints:
- joint hip_pitch_servo: origin xyz=0 0 0 -> xyz=-0.00991 0.01295 0.001005 rpy=0 -1.57079632679 3.1415927
- joint hip_yaw_servo: origin xyz=0 0 0 -> xyz=0 -0.00995 0 rpy=0 0 0
- joint left_front_pitch_swivel: origin xyz=-0.01035 -0.00995 0.0292 -> xyz=-0.01035 0 0.0292 rpy=3.1415927 0 -1.57079632679
- joint swivel: origin xyz=-0.01035 -0.00995 0.0292 -> xyz=-0.01035 0 0.0292 rpy=3.1415927 0 -1.57079632679

Commit message: Adding thigh

File: src/servo/urdf/servo.urdf (robot description, URDF)
Before this commit: robot servo, 5 links, 4 joints
Links:
- added link left_front_thigh; visual mesh filename=package://servo/meshes/Thigh_V15.stl scale=0.001 0.001 0.001
Joints:
- added joint left_front_thigh: type fixed, parent left_front_pitch_servo_horn, child left_front_thigh, origin xyz=0 0 0 rpy=1.5707963 0 0

Commit message: Adding knee servo horn

File: src/servo/urdf/servo.urdf (robot description, URDF)
Before this commit: robot hexapod, 6 links, 5 joints
Links:
- added link left_front_knee_servo_horn; visual mesh filename=package://servo/meshes/ServoHorn.stl
Joints:
- added joint left_front_knee: type fixed, parent left_front_thigh, child left_front_knee_servo_horn, origin xyz=0.080 0 0 rpy=-1.5707963 3.1415927 0

Commit message: Adding knee servo

File: src/servo/urdf/servo.urdf (robot description, URDF)
Before this commit: robot hexapod, 7 links, 6 joints
Links:
- added link left_front_knee_servo_base; visual mesh filename=package://servo/meshes/Servo.stl
Joints:
- added joint left_front_knee_swivel: type continuous, parent left_front_knee_servo_horn, child left_front_knee_servo_base, origin xyz=0 -0.01035 0.0292 rpy=3.1415927 0 -1.5707963, axis 0 0 -1

Commit message: Adding Shin to URDF

File: src/servo/urdf/servo.urdf (robot description, URDF)
Before this commit: robot hexapod, 8 links, 7 joints
Links:
- added link left_front_shin; visual mesh filename=package://servo/meshes/LeftShin_V15.stl scale=0.001 0.001 0.001
Joints:
- added joint left_front_shin: type fixed, parent left_front_knee_servo_base, child left_front_shin, origin xyz=0 -0.00995 0 rpy=-1.5707963 0 0

Commit message: Adding Body as new top level link

File: src/servo/urdf/servo.urdf (robot description, URDF)
Before this commit: robot hexapod, 9 links, 8 joints
Links:
- added link body_top; visual mesh filename=package://servo/meshes/BodyTop_V16.stl scale=0.001 0.001 0.001
Joints:
- added joint body_to_front_left: type fixed, parent body_top, child left_front_yaw_servo_horn, origin xyz=0 0 0.0045 rpy=3.1415927 0 -1.5707963
- joint hip_yaw_servo: child left_front_yaw_servo_base -> left_hip; origin xyz=0 -0.00995 0 rpy=0 0 0 -> xyz=0 0.00995 0 rpy=0 0 0; parent left_hip -> left_front_yaw_servo_base
- joint swivel: child left_front_yaw_servo_horn -> left_front_yaw_servo_base; origin xyz=-0.01035 0 0.0292 rpy=3.1415927 0 -1.57079632679 -> xyz=0 -0.01035 0.0292 rpy=0 3.1415927 1.5707963; parent left_front_yaw_servo_base -> left_front_yaw_servo_horn

Commit message: Adding body bottom and center, and fixing position of yaw servo

File: src/servo/urdf/servo.urdf (robot description, URDF)
Before this commit: robot hexapod, 10 links, 9 joints
Links:
- added link body_bottom; visual mesh filename=package://servo/meshes/BodyBottom_V16.stl scale=0.001 0.001 0.001
- added link body_center; visual mesh filename=package://servo/meshes/CenterStrut_V16.stl scale=0.001 0.001 0.001
Joints:
- added joint body_top_to_bottom: type fixed, parent body_top, child body_bottom, origin xyz=0 0 0
- added joint body_top_to_center: type fixed, parent body_top, child body_center, origin xyz=0 0 0
- joint body_to_front_left: origin xyz=0 0 0.0045 rpy=3.1415927 0 -1.5707963 -> xyz=0 0 0.005 rpy=3.1415927 0 -1.5707963
- joint hip_yaw_servo: origin xyz=0 0.00995 0 rpy=0 0 0 -> xyz=0.01035 0.00995 -0.0292
- joint swivel: origin xyz=0 -0.01035 0.0292 rpy=0 3.1415927 1.5707963 -> xyz=0 0 0 rpy=0 3.1415927 1.5707963

Commit message: Fixing Shin connection

File: src/servo/urdf/servo.urdf (robot description, URDF)
Before this commit: robot hexapod, 12 links, 11 joints
Joints:
- joint left_front_knee_swivel: origin xyz=0 -0.01035 0.0292 rpy=3.1415927 0 -1.5707963 -> xyz=0 0 0 rpy=3.1415927 0 -1.5707963
- joint left_front_shin: origin xyz=0 -0.00995 0 rpy=-1.5707963 0 0 -> xyz=0.01035 -0.00995 -0.02889 rpy=-1.5707963 0 0
